Commit message: updates

File: data/o2/o2.urdf (robot description, URDF)
Before this commit: robot panda, 37 links, 36 joints
Joints:
- removed joint base_joint6f
- removed joint base_joint6f1
- removed joint left_joint2f
- removed joint left_joint3f
- removed joint left_joint4f
- removed joint left_joint5f
- removed joint left_joint8
- removed joint left_joint8f
- removed joint left_joint_chassis
- removed joint right_joint2f
- removed joint right_joint3f
- removed joint right_joint4f
- removed joint right_joint5f
- removed joint right_joint8
- removed joint right_joint8f
- removed joint right_joint_chassis
- added joint base_fixed6f: type fixed, parent base_link6, child base_link6f, origin xyz=0 0 0 rpy=0 0 0, axis 0 0 1, limit lower=-2.8973 upper=2.8973 effort=87 velocity=2.1750
- added joint base_fixed6f1: type fixed, parent base_link6f, child base_link6f1, origin xyz=0 0 0 rpy=0 0 0, axis 0 0 1, limit lower=-2.8973 upper=2.8973 effort=87 velocity=2.1750
- added joint left_fixed2f: type fixed, parent left_link2, child left_link2f, origin xyz=0 0 0 rpy=0 0 0, axis 0 0 1, limit lower=-2.8973 upper=2.8973 effort=87 velocity=2.1750
- added joint left_fixed3f: type fixed, parent left_link3, child left_link3f, origin xyz=0 0 0 rpy=0 0 0, axis 0 0 1, limit lower=-2.8973 upper=2.8973 effort=87 velocity=2.1750
- added joint left_fixed4f: type fixed, parent left_link4, child left_link4f, origin xyz=0 0 0 rpy=0 0 0, axis 0 0 1, limit lower=-2.8973 upper=2.8973 effort=87 velocity=2.1750
- added joint left_fixed5f: type fixed, parent left_link5, child left_link5f, origin xyz=0 0 0 rpy=0 0 0, axis 0 0 1, limit lower=-2.8973 upper=2.8973 effort=87 velocity=2.1750
- added joint left_fixed8: type fixed, parent left_link7, child left_link8, origin xyz=0 -0.23675 0 rpy=1.5707963 0 0, axis 0 0 1, limit lower=-2.8973 upper=2.8973 effort=87 velocity=2.1750
- added joint left_fixed8f: type fixed, parent left_link8, child left_link8f, origin xyz=0 0 0 rpy=0 0 0, axis 0 0 1, limit lower=-2.8973 upper=2.8973 effort=87 velocity=2.1750
- added joint left_fixed_chassis: type fixed, parent base_link6, child left_chassis, origin xyz=0.58 0.2 0 rpy=0 0 -0.785398, axis 0 0 1, limit lower=-2.8973 upper=2.8973 effort=87 velocity=2.1750
- added joint right_fixed2f: type fixed, parent right_link2, child right_link2f, origin xyz=0 0 0 rpy=0 0 0, axis 0 0 1, limit lower=-2.8973 upper=2.8973 effort=87 velocity=2.1750
- added joint right_fixed3f: type fixed, parent right_link3, child right_link3f, origin xyz=0 0 0 rpy=0 0 0, axis 0 0 1, limit lower=-2.8973 upper=2.8973 effort=87 velocity=2.1750
- added joint right_fixed4f: type fixed, parent right_link4, child right_link4f, origin xyz=0 0 0 rpy=0 0 0, axis 0 0 1, limit lower=-2.8973 upper=2.8973 effort=87 velocity=2.1750
- added joint right_fixed5f: type fixed, parent right_link5, child right_link5f, origin xyz=0 0 0 rpy=0 0 0, axis 0 0 1, limit lower=-2.8973 upper=2.8973 effort=87 velocity=2.1750
- added joint right_fixed8: type fixed, parent right_link7, child right_link8, origin xyz=0 -0.23675 0 rpy=1.5707963 0 0, axis 0 0 1, limit lower=-2.8973 upper=2.8973 effort=87 velocity=2.1750
- added joint right_fixed8f: type fixed, parent right_link8, child right_link8f, origin xyz=0 0 0 rpy=0 0 0, axis 0 0 1, limit lower=-2.8973 upper=2.8973 effort=87 velocity=2.1750
- added joint right_fixed_chassis: type fixed, parent base_link6, child right_chassis, origin xyz=0.58 -0.2 0 rpy=0 0 0.785398, axis 0 0 1, limit lower=-2.8973 upper=2.8973 effort=87 velocity=2.1750

Commit message: Flexible joint

File: data/o2/o2.urdf (robot description, URDF)
Before this commit: robot panda, 37 links, 36 joints
Links:
- added link left_sensor, mass 0.001; collision box size=0.1 0.1 0.1; visual box size=0.1 0.1 0.1
Joints:
- added joint left_fixed_sensor: type fixed, parent left_link8, child left_sensor, origin xyz=0 0 0 rpy=0 0 0, axis 0 0 1, limit lower=-2.8973 upper=2.8973 effort=87 velocity=2.1750
